Commit message: DWA algorithm implemented, next step collision avoidance

File: urdf/ugv_rviz.xacro (robot description, xacro)
@@ -17,6 +17,8 @@
   <!-- Import Rviz colors -->
   <!-- <xacro:include filename="$(find testing)/urdf/materials.xacro" /> -->
-  <!-- Used for fixing robot to Gazebo 'base_link' -->
-  <link name="odom"/>
+  <!-- fixed odom  -->
+  <link name="odom">
+    <origin xyz="0 0 0" rpy="0 0 0"/>
+  </link>
   <joint name="footprint_joint" type="fixed">
     <origin xyz="0 0 0" rpy="0 0 0"/>
